File: HARDWARE/OPAM UAA/OPAM UAA.sch (KiCad schematic (older format))
At the start: 20 parts, among them J1 BATT+, J2 CELDA, U1 LM317L_TO92, U2 LM324A, U3 LM35-LP, U4 LM35-LP

Commit message: PCB 2.0
Parts:
- added J3: salida1, Pin_Headers:Pin_Header_Straight_1x02_Pitch2.54mm, symbol conn:Conn_01x02
- added J4: salida2, Pin_Headers:Pin_Header_Straight_1x02_Pitch2.54mm, symbol conn:Conn_01x02
- added R14, R15: 8.2K, Resistors_THT:R_Axial_DIN0411_L9.9mm_D3.6mm_P12.70mm_Horizontal, symbol device:R
- J1, J2: footprint (none) -> Pin_Headers:Pin_Header_Straight_1x02_Pitch2.54mm
- R1, R2, R3, R4, R5, R6, R7, R8, R9: footprint (none) -> Resistors_THT:R_Axial_DIN0411_L9.9mm_D3.6mm_P12.70mm_Horizontal
- R10, R12: value R -> 47K; footprint (none) -> Resistors_THT:R_Axial_DIN0411_L9.9mm_D3.6mm_P12.70mm_Horizontal
- R11, R13: value R -> 180K; footprint (none) -> Resistors_THT:R_Axial_DIN0411_L9.9mm_D3.6mm_P12.70mm_Horizontal
- RV1: footprint (none) -> Potentiometers:Potentiometer_WirePads_largePads
- U1: footprint TO_SOT_Packages_THT:TO-92_Inline_Narrow_Oval -> TO_SOT_Packages_THT:TO-92_Inline_Wide
- U2: footprint (none) -> Housings_DIP:DIP-14_W7.62mm_Socket_LongPads
- U3, U4: footprint (none) -> TO_SOT_Packages_THT:TO-92_Inline_Narrow_Oval
Connections:
- net GND: now also J3.1 (Pin_1), J4.1 (Pin_1)
- net at R11.1: now also R14.2; no longer U2.8
- net at R13.1: now also R15.2; no longer U2.14
- new net salida1: J3.2 (Pin_2), R14.1, U2.8
- new net salida2: J4.2 (Pin_2), R15.1, U2.14
Other:
- moved on the sheet: R10, R11, R12, R13, U2D, U4

Commit message: BUGS 2.0
Parts:
- removed R6: 1K, Resistors_THT:R_Axial_DIN0411_L9.9mm_D3.6mm_P12.70mm_Horizontal, symbol device:R
- added CON-CELDA1: Conn_01x02, symbol conn:Conn_01x02
- R2: value R -> 330
- R4: value 12K -> 8.2K
- renumbered R1 to 1.2K1
Connections:
- net GND: now also R5.2, CON-CELDA1.1 (Pin_1)
- net SALIDA-CELDA: now reaches RV1.2, RV1.3, U2.7
- net SALIDA-CELDA: now also CON-CELDA1.2 (Pin_2)
Changed lines of the file:
@@
 $EndComp
 $Comp
-L device:R R1
+L device:R 1.2K1
 U 1 1 5D071FDD
 P 1200 1500
-F 0 "R1" H 1270 1546 50  0000 L CNN
+F 0 "1.2K1" H 1270 1546 50  0000 L CNN
 F 1 "R" H 1270 1455 50  0000 L CNN
 F 2 "Resistors_THT:R_Axial_DIN0411_L9.9mm_D3.6mm_P12.70mm_Horizontal" V 1130 1500 50  0001 C CNN
@@
 P 1500 1300
 F 0 "R2" V 1293 1300 50  0000 C CNN
-F 1 "R" V 1384 1300 50  0000 C CNN
+F 1 "330" V 1384 1300 50  0000 C CNN
 F 2 "Resistors_THT:R_Axial_DIN0411_L9.9mm_D3.6mm_P12.70mm_Horizontal" V 1430 1300 50  0001 C CNN
 F 3 "~" H 1500 1300 50  0001 C CNN
@@
 $EndComp
 Wire Wire Line
-	3550 2150 3550 2350
-Wire Wire Line
 	3550 1650 3550 1850
-$Comp
-L device:R R6
-U 1 1 5D070005
-P 3550 2500
-F 0 "R6" H 3620 2546 50  0000 L CNN
-F 1 "1K" H 3620 2455 50  0000 L CNN
-F 2 "Resistors_THT:R_Axial_DIN0411_L9.9mm_D3.6mm_P12.70mm_Horizontal" V 3480 2500 50  0001 C CNN
-F 3 "~" H 3550 2500 50  0001 C CNN
-	1    3550 2500
-	1    0    0    -1
-$EndComp
 $Comp
 L device:R R5
@@
 P 3550 1500
 F 0 "R4" H 3620 1546 50  0000 L CNN
-F 1 "12K" H 3620 1455 50  0000 L CNN
+F 1 "8.2K" H 3620 1455 50  0000 L CNN
 F 2 "Resistors_THT:R_Axial_DIN0411_L9.9mm_D3.6mm_P12.70mm_Horizontal" V 3480 1500 50  0001 C CNN
 F 3 "~" H 3550 1500 50  0001 C CNN
@@
 	5400 1350 5650 1350
 Wire Wire Line
-	5650 1350 5650 1800
+	5650 1350 5650 1500
 Connection ~ 5650 1800
 Wire Wire Line
@@
 L power:GND #PWR05
 U 1 1 5D075C8E
-P 3550 2750
-F 0 "#PWR05" H 3550 2500 50  0001 C CNN
-F 1 "GND" H 3555 2577 50  0000 C CNN
-F 2 "" H 3550 2750 50  0001 C CNN
-F 3 "" H 3550 2750 50  0001 C CNN
-	1    3550 2750
-	1    0    0    -1
-$EndComp
-Wire Wire Line
-	3550 2650 3550 2750
+P 3550 2450
+F 0 "#PWR05" H 3550 2200 50  0001 C CNN
+F 1 "GND" H 3555 2277 50  0000 C CNN
+F 2 "" H 3550 2450 50  0001 C CNN
+F 3 "" H 3550 2450 50  0001 C CNN
+	1    3550 2450
+	1    0    0    -1
+$EndComp
 $Comp
 L power:GND #PWR06
@@
 Wire Notes Line
 	6150 3550 6150 550
-Text Notes 4300 3150 0    118  ~ 24
+Text Notes 3300 3150 0    118  ~ 24
 ETAPA DE\nCONTROL 1
 Wire Notes Line
@@
 Wire Wire Line
 	7550 1400 7550 2150
-Wire Wire Line
-	10050 1500 10050 2200
 $Comp
 L device:R R14
@@
 Wire Notes Line
 	8700 500  8700 3550
+Wire Wire Line
+	10050 1500 10050 2200
+Wire Wire Line
+	3550 2150 3550 2450
+$Comp
+L conn:Conn_01x02 CON-CELDA1
+U 1 1 5D095DE8
+P 4900 3000
+F 0 "CON-CELDA1" H 4820 2675 50  0000 C CNN
+F 1 "Conn_01x02" H 4820 2766 50  0000 C CNN
+F 2 "" H 4900 3000 50  0001 C CNN
+F 3 "~" H 4900 3000 50  0001 C CNN
+	1    4900 3000
+	-1   0    0    1
+$EndComp
+Text Label 5700 1500 0    39   ~ 0
+SALIDA-CELDA
+Wire Wire Line
+	5700 1500 5650 1500
+Connection ~ 5650 1500
+Wire Wire Line
+	5650 1500 5650 1800
+Text Label 5250 2900 0    39   ~ 0
+SALIDA-CELDA
+Wire Wire Line
+	5100 2900 5250 2900
+$Comp
+L power:GND #PWR014
+U 1 1 5D0998F5
+P 5300 3000
+F 0 "#PWR014" H 5300 2750 50  0001 C CNN
+F 1 "GND" H 5305 2827 50  0000 C CNN
+F 2 "" H 5300 3000 50  0001 C CNN
+F 3 "" H 5300 3000 50  0001 C CNN
+	1    5300 3000
+	1    0    0    -1
+$EndComp
+Wire Wire Line
+	5100 3000 5300 3000
 $EndSCHEMATC

Commit message: BUGS 3.0
Parts:
- 1.2K1: value R -> R1
- CON-CELDA1: footprint (none) -> Pin_Headers:Pin_Header_Straight_1x02_Pitch2.54mm
Changed lines of the file:
@@
 P 1200 1500
 F 0 "1.2K1" H 1270 1546 50  0000 L CNN
-F 1 "R" H 1270 1455 50  0000 L CNN
+F 1 "R1" H 1270 1455 50  0000 L CNN
 F 2 "Resistors_THT:R_Axial_DIN0411_L9.9mm_D3.6mm_P12.70mm_Horizontal" V 1130 1500 50  0001 C CNN
 F 3 "~" H 1200 1500 50  0001 C CNN
@@
 F 0 "CON-CELDA1" H 4820 2675 50  0000 C CNN
 F 1 "Conn_01x02" H 4820 2766 50  0000 C CNN
-F 2 "" H 4900 3000 50  0001 C CNN
+F 2 "Pin_Headers:Pin_Header_Straight_1x02_Pitch2.54mm" H 4900 3000 50  0001 C CNN
 F 3 "~" H 4900 3000 50  0001 C CNN
 	1    4900 3000
