File: HARDWARE/OPAM UAA/OPAM UAA.kicad_pcb (KiCad board)
At the start: 2 copper layers, 99.1 x 50.8 mm, 24 parts, among them J1 BATT+, J2 CELDA, J3 salida1, J4 salida2, U1 LM317L_TO92, U2 LM324A, U3 LM35-LP, U4 LM35-LP

Commit message: BUGS
Parts:
- renumbered J1 to BATT, J2 to CELDA, J3 to SALIDA1, J4 to SALIDA4
Routing:
- net /VCC-REGULADOR: track 92.9 -> 91.9 mm
Changed lines of the file:
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@@
     (thickness 1.6)
     (drawings 4)
-    (tracks 153)
+    (tracks 154)
     (zones 0)
     (modules 24)
@@
     (descr "Through hole straight pin header, 1x02, 2.54mm pitch, single row")
     (tags "Through hole pin header THT 1x02 2.54mm single row")
-    (fp_text reference J1 (at 0 -2.33 180) (layer F.SilkS)
+    (fp_text reference BATT (at 0 -2.33 180) (layer F.SilkS)
       (effects (font (size 1 1) (thickness 0.15)))
     )
@@
     (descr "Through hole straight pin header, 1x02, 2.54mm pitch, single row")
     (tags "Through hole pin header THT 1x02 2.54mm single row")
-    (fp_text reference J2 (at 0 -2.33 180) (layer F.SilkS)
+    (fp_text reference CELDA (at 0 -2.33 180) (layer F.SilkS)
       (effects (font (size 1 1) (thickness 0.15)))
     )
@@
     (descr "Through hole straight pin header, 1x02, 2.54mm pitch, single row")
     (tags "Through hole pin header THT 1x02 2.54mm single row")
-    (fp_text reference J3 (at 0 -2.33) (layer F.SilkS)
+    (fp_text reference SALIDA1 (at 0 -2.33) (layer F.SilkS)
       (effects (font (size 1 1) (thickness 0.15)))
     )
@@
     (descr "Through hole straight pin header, 1x02, 2.54mm pitch, single row")
     (tags "Through hole pin header THT 1x02 2.54mm single row")
-    (fp_text reference J4 (at 0 -2.33 180) (layer F.SilkS)
+    (fp_text reference SALIDA4 (at 0 -2.33 180) (layer F.SilkS)
       (effects (font (size 1 1) (thickness 0.15)))
     )
@@
   (segment (start 124.425011 99.149999) (end 128.842989 99.149999) (width 1.3) (layer B.Cu) (net 6))
   (segment (start 130.02299 104.779989) (end 128.909989 105.89299) (width 1.3) (layer B.Cu) (net 6))
+  (segment (start 158.75 123.23) (end 158.75 125.73) (width 1.3) (layer B.Cu) (net 7))
+  (segment (start 112.300021 122.460021) (end 157.980021 122.460021) (width 1.3) (layer B.Cu) (net 7))
+  (segment (start 157.980021 122.460021) (end 158.75 123.23) (width 1.3) (layer B.Cu) (net 7))
+  (segment (start 127 104.100002) (end 122.410001 108.690001) (width 1.3) (layer B.Cu) (net 7))
+  (segment (start 122.410001 108.690001) (end 118.889999 108.690001) (width 1.3) (layer B.Cu) (net 7))
   (segment (start 118.889999 108.690001) (end 115.169999 104.970001) (width 1.3) (layer B.Cu) (net 7))
-  (segment (start 112.300021 122.460021) (end 157.980021 122.460021) (width 1.3) (layer B.Cu) (net 7))
-  (segment (start 158.75 123.23) (end 158.75 125.73) (width 1.3) (layer B.Cu) (net 7))
   (segment (start 108.389999 118.549999) (end 112.300021 122.460021) (width 1.3) (layer B.Cu) (net 7))
-  (segment (start 127 104.100002) (end 122.410001 108.690001) (width 1.3) (layer B.Cu) (net 7))
-  (segment (start 157.980021 122.460021) (end 158.75 123.23) (width 1.3) (layer B.Cu) (net 7))
-  (segment (start 122.410001 108.690001) (end 118.889999 108.690001) (width 1.3) (layer B.Cu) (net 7))
-  (segment (start 108.389999 104.970001) (end 108.389999 118.549999) (width 1.3) (layer B.Cu) (net 7))
-  (segment (start 115.169999 104.970001) (end 108.389999 104.970001) (width 1.3) (layer B.Cu) (net 7))
-  (segment (start 127 104.100002) (end 127 101.6) (width 1.3) (layer B.Cu) (net 7))
+  (segment (start 115.169999 104.970001) (end 110.099998 104.970001) (width 1.3) (layer B.Cu) (net 7))
+  (segment (start 108.389999 106.68) (end 108.389999 118.549999) (width 1.3) (layer B.Cu) (net 7))
+  (segment (start 127 101.6) (end 127 104.100002) (width 1.3) (layer B.Cu) (net 7))
+  (segment (start 110.099998 104.970001) (end 108.389999 106.68) (width 1.3) (layer B.Cu) (net 7))
   (segment (start 132.08 134.62) (end 137.16 134.62) (width 1.3) (layer B.Cu) (net 8))
   (segment (start 141.510012 130.269988) (end 154.170012 130.269988) (width 1.3) (layer B.Cu) (net 8))

Commit message: BUGS 3.0
Parts:
- removed BATT: BATT+, Pin_Headers:Pin_Header_Straight_1x02_Pitch2.54mm
- removed CELDA: CELDA, Pin_Headers:Pin_Header_Straight_1x02_Pitch2.54mm
- removed R1: R, Resistors_THT:R_Axial_DIN0411_L9.9mm_D3.6mm_P12.70mm_Horizontal
- removed SALIDA1: salida1, Pin_Headers:Pin_Header_Straight_1x02_Pitch2.54mm
- removed SALIDA4: salida2, Pin_Headers:Pin_Header_Straight_1x02_Pitch2.54mm
- added 1.2K1: R1, Resistors_THT:R_Axial_DIN0411_L9.9mm_D3.6mm_P12.70mm_Horizontal, F.Cu at (127.0, 116.8)
- added CON-CELDA1: Conn_01x02, Pin_Headers:Pin_Header_Straight_1x02_Pitch2.54mm, F.Cu at (198.1, 117.5)
- added J1: BATT+, Pin_Headers:Pin_Header_Straight_1x02_Pitch2.54mm, F.Cu at (110.5, 110.5)
- added J2: CELDA, Pin_Headers:Pin_Header_Straight_1x02_Pitch2.54mm, F.Cu at (110.5, 138.4)
- added J3: salida1, Pin_Headers:Pin_Header_Straight_1x02_Pitch2.54mm, F.Cu at (198.1, 104.1)
- added J4: salida2, Pin_Headers:Pin_Header_Straight_1x02_Pitch2.54mm, F.Cu at (198.1, 129.5)
- R2: value R -> 330
- R4: value 12K -> 8.2K
Connections:
- net Net-(RV1-Pad2) renamed /SALIDA-CELDA
- R5 pad 2: Net-(R5-Pad2) -> GND
Routing:
- net /SALIDA-CELDA: track 27.6 -> 53.2 mm

Commit message: PCB 3.0
Parts:
- removed R6: 1K, Resistors_THT:R_Axial_DIN0411_L9.9mm_D3.6mm_P12.70mm_Horizontal
- moved 1.2K1 107.8 mm to (50.8, 40.6)
- moved J2 107.8 mm to (34.3, 62.2)
- moved J3 107.8 mm to (121.9, 27.9)
- moved R11 107.8 mm to (109.6, 39.3)
- moved R15 107.8 mm to (69.8, 39.4)
- moved R5 107.8 mm to (73.7, 66.0)
- moved R9 107.8 mm to (96.5, 66.0)
- moved RV1 107.8 mm to (101.6, 58.4)
- moved U1 107.8 mm to (44.5, 30.5)
- moved CON-CELDA1 107.8 mm to (121.9, 41.3)
- moved J4 107.8 mm to (121.9, 53.3)
- moved R12 107.8 mm to (88.9, 27.9)
- moved R14 107.8 mm to (96.9, 33.0)
- moved R2 107.8 mm to (50.8, 25.4)
- moved R3 107.8 mm to (43.2, 58.4)
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Routing:
- net GND: track 22.9 -> 31.1 mm, vias 6 -> 8
- net Net-(R5-Pad2): track 5.08 -> 0.00 mm
Other:
- net class Default: clearance 0.6 -> 0.2; trace_width 1.3 -> 0.6
- rule trace_clearance: 0.6 -> 0.2
- board text added: "INGENIERIA EN ENERGIAS RENOVABLES"
